File: Final schematic/Final schematic.kicad_pcb (KiCad board)
At the start: 2 copper layers, 140 x 90 mm, 38 parts, among them J1 PJ-102AH, J2 Conn_01x06, J3 Conn_02x03_Odd_Even, SW1 Omron_B3F_SPST, SW2 Omron_B3F_SPST, SW3 Omron_B3F_SPST, SW4 Omron_B3F_SPST, U1 ATmega328-PU, U3 MAX7219, U4 DS1307_DIP-8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

Commit message: pdb update
Parts:
- moved C4 180.7 mm to (124.5, 78.7)
- moved C9 171.2 mm to (124.5, 71.1)
- moved C5 147.6 mm to (124.5, 83.8), turned to 180 degrees
- moved R3 143.2 mm to (137.2, 66.0)
- moved C3 138.0 mm to (195.6, 73.7)
- moved C2 133.1 mm to (205.7, 91.4)
- moved R10 132.4 mm to (129.5, 137.2), turned to 180 degrees
- moved C8 128.4 mm to (124.5, 74.5), turned to 180 degrees
- moved C6 120.1 mm to (157.5, 86.4), turned to 180 degrees
- moved R5 119.4 mm to (142.2, 66.0)
- moved R6 117.0 mm to (149.9, 121.9), turned to 180 degrees
- moved R8 115.1 mm to (149.9, 137.2)
- moved C7 95.5 mm to (172.7, 81.3)
- moved R7 80.5 mm to (170.2, 137.2)
- moved C1 80.2 mm to (154.9, 66.0)
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
Commit message: pcb update
Parts:
- added C9: C_0805_10uf, footprints:C_0805_2012Metric, F.Cu at (186.7, 47.0)
- moved J2 26.1 mm to (191.8, 96.5)
- moved C2 19.7 mm to (197.3, 109.2)
- moved R4 15.3 mm to (194.3, 69.8), turned to 90 degrees
- moved C7 13.1 mm to (161.3, 87.6)
- moved J1 9.25 mm to (201.9, 68.6)
- moved C3 8.57 mm to (203.6, 76.6)
- moved Y1 4.02 mm to (158.8, 82.5)
- moved R6 3.81 mm to (149.9, 125.7)
- moved DS1 3.17 mm to (152.4, 100.3)
- moved SW2 2.54 mm to (170.2, 132.1)
- moved SW3 2.54 mm to (149.9, 132.1)
- moved SW4 2.54 mm to (129.5, 132.1)
- moved R10 2.54 mm to (129.5, 139.7)
- moved R7 2.54 mm to (170.2, 139.7)
- moved R8 2.54 mm to (149.9, 139.7)
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Routing:
- net Net-(C7-Pad1): track 0.00 -> 11.9 mm
- net Net-(C6-Pad1): track 0.00 -> 11.8 mm
- net GND: track 0.00 -> 3.38 mm, vias 0 -> 2
- added copper zone on B.Cu, net GND
- added copper zone on F.Cu, net VCC

Commit message: pcb update
Parts:
- removed the C9 at (124.5, 72.4)
- added U2: L7805, footprints:TO-252-2, F.Cu at (205.7, 80.0)
- moved C9 85.1 mm to (156.2, 126.5)
- moved C5 77.5 mm to (201.9, 85.1)
- moved C8 63.4 mm to (162.6, 126.5)
- moved R10 38.6 mm to (168.1, 141.2)
- moved SW4 38.6 mm to (168.1, 133.6)
- moved R7 36.9 mm to (133.3, 141.2)
- moved SW2 36.1 mm to (134.1, 133.3)
- moved C4 29.3 mm to (153.7, 82.5)
- moved BT1 28.6 mm to (87.4, 125.7), turned to 0 degrees
- moved R4 14.6 mm to (180.3, 65.6)
- moved C7 6.88 mm to (168.1, 88.9)
- moved C6 6.88 mm to (163.0, 88.9)
- moved Y1 6.48 mm to (165.1, 83.8)
- moved C3 2.65 mm to (205.7, 74.9)
- moved J1 2.54 mm to (204.5, 68.6)
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Routing:
- net BTN_UP: track 0.00 -> 128.8 mm
- net BTN_SEL: track 0.00 -> 112.8 mm
- net BTN_DWN: track 0.00 -> 100.2 mm
- net GND: track 3.38 -> 89.2 mm, vias 2 -> 19
- net Net-(J2-Pad5): track 0.00 -> 69.5 mm
- net RESET: track 0.00 -> 68.2 mm
- net Net-(J2-Pad4): track 0.00 -> 62.6 mm
- net VCC: track 0.00 -> 54.3 mm
- net SDA: track 0.00 -> 54.2 mm
- net SCL: track 0.00 -> 46.8 mm
- net Net-(BT1-Pad1): track 0.00 -> 44.3 mm
- net MOSI: track 0.00 -> 17.2 mm
- net MISO: track 0.00 -> 14.7 mm
- net LED_SCK: track 0.00 -> 8.79 mm
- net Net-(C3-Pad1): track 0.00 -> 8.03 mm
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
Commit message: pcb update
Routing:
- net DISP_CLK: track 0.00 -> 101.0 mm
- net DISP_LOAD: track 0.00 -> 74.9 mm
- net Net-(DS1-Pad12): track 0.00 -> 69.8 mm, vias 0 -> 1
- net Net-(DS1-Pad13): track 0.00 -> 68.5 mm
- net DISP_DATA: track 0.00 -> 61.2 mm
- net Net-(DS1-Pad14): track 0.00 -> 60.4 mm, vias 0 -> 1
- net Net-(DS1-Pad2): track 0.00 -> 55.6 mm
- net Net-(DS1-Pad1): track 0.00 -> 49.6 mm
- net Net-(DS1-Pad3): track 0.00 -> 41.6 mm, vias 0 -> 1
- net Net-(DS1-Pad9): track 0.00 -> 35.5 mm, vias 0 -> 1
- net RESET: track 68.2 -> 102.6 mm
- net Net-(DS1-Pad11): track 0.00 -> 26.1 mm
- net Net-(DS1-Pad10): track 0.00 -> 21.9 mm
- net Net-(DS1-Pad5): track 0.00 -> 21.1 mm
- net Net-(DS1-Pad6): track 0.00 -> 13.5 mm, vias 0 -> 1
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