File: Final schematic/Final schematic.kicad_pcb (KiCad board)
At the start: 2 copper layers, 140 x 90 mm, 39 parts, among them J1 Power_inlet_vertical, J2 Conn_01x06, J3 Conn_02x03_Odd_Even, SW1 Omron_B3F_SPST, SW2 Omron_B3F_SPST, SW3 Omron_B3F_SPST, SW4 Omron_B3F_SPST, U1 ATmega328-PU, U2 L7805, U3 MAX7219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

Commit message: gerber out
Other:
- board text added: "The GG-Board"
Changed lines of the file:
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@@
     )
     (pad_to_mask_clearance 0)
+    (aux_axis_origin 78.74 144.78)
     (pcbplotparams
       (layerselection 0x00010fc_ffffffff)
@@
   (gr_line locked (start 210.6 57) (end 150 57) (layer "User.4") (width 0.05))
   (gr_line locked (start 82 64.4) (end 85 64.4) (layer "User.4") (width 0.05))
+  (gr_text "The GG-Board" (at 195.58 137.16) (layer "F.SilkS")
+    (effects (font (size 2 2) (thickness 0.15)))
+  )
   (segment (start 97.8 97.8) (end 86.604 97.8) (width 0.3048) (layer "F.Cu") (net 1))
   (segment (start 83.82 100.584) (end 83.82 125.984) (width 0.3048) (layer "F.Cu") (net 1))
