File: Final schematic/_autosave-Final schematic.kicad_pcb (KiCad board)
At the start: 2 copper layers, 140 x 90 mm, 39 parts, among them J1 PJ-102AH, J2 Conn_01x06, J3 Conn_02x03_Odd_Even, SW1 Omron_B3F_SPST, SW2 Omron_B3F_SPST, SW3 Omron_B3F_SPST, SW4 Omron_B3F_SPST, U1 ATmega328-PU, U2 L7805, U3 MAX7219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

Commit message: pcb update
pcb update
Parts:
- removed C3: C_0805_0.1uf, footprints:C_0805_2012Metric
- DS1: value LED_Display_1001 -> LED
- J1: value PJ-102AH -> VAL**
Routing:
- net GND: track 96.1 -> 75.3 mm
- net VCC: track 54.3 -> 66.5 mm, vias 0 -> 11
- net Net-(C3-Pad1): track 8.03 -> 7.36 mm
