File: Final schematic/_autosave-Final schematic.kicad_sch (KiCad schematic)
At the start: 39 parts, among them J1 PJ-102AH, J2 Conn_01x06, J3 Conn_02x03_Odd_Even, SW1 Omron_B3F_SPST, SW2 Omron_B3F_SPST, SW3 Omron_B3F_SPST, SW4 Omron_B3F_SPST, U1 ATmega328-PU, U2 L7805, U3 MAX7219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

Commit message: PCB UPDATE
Parts:
- removed J1: PJ-102AH, footprints:PJ-102AH, symbol HPS:PJ-102AH
- added J1: Power_inlet_vertical, footprints:Wurth-694106402002, symbol HPS:Power_inlet_vertical
Connections:
- net GND: now also J1.2 (OUT)
- net at C3.1, U2.1 (IN): now also J1.1 (POLE)
Changed lines of the file:
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@@
     )
-  )
-  (symbol (lib_id "HPS:PJ-102AH") (at 26.67 134.62 0) (unit 1)
-    (in_bom yes) (on_board yes) (fields_autoplaced)
-    (property "Reference" "J1" (id 0) (at 24.13 121.92 0)
-      (effects (font (size 1.524 1.524)))
-    )
-    (property "Value" "PJ-102AH" (id 1) (at 24.13 125.73 0)
-      (effects (font (size 1.524 1.524)))
-    )
-    (property "Footprint" "footprints:PJ-102AH" (id 2) (at 24.13 129.54 0)
-      (effects (font (size 1.524 1.524)))
-    )
-    (property "Datasheet" "https://www.cuidevices.com/product/resource/pj-102ah.pdf" (id 3) (at 28.194 146.558 0)
-      (effects (font (size 1.524 1.524)) hide)
-    )
-    (property "MFG" "CUI Devices" (id 4) (at 26.67 152.4 0)
-      (effects (font (size 1.27 1.27)) hide)
-    )
-    (property "MPN" "PJ-102AH" (id 5) (at 26.67 154.94 0)
-      (effects (font (size 1.27 1.27)) hide)
-    )
-    (property "Digikey PN" "CP-102AH-ND" (id 6) (at 28.194 160.147 0)
-      (effects (font (size 1.27 1.27)) hide)
-    )
-    (property "Mouser PN" "490-PJ-102AH" (id 7) (at 26.67 157.353 0)
-      (effects (font (size 1.27 1.27)) hide)
-    )
-    (pin "1")
-    (pin "2")
-    (pin "3")
   )
   (symbol (lib_id "HPS:MAX7219") (at 140.97 62.23 0) (unit 1)
@@
     (pin "1")
   )
+  (symbol (lib_id "HPS:Power_inlet_vertical") (at 26.67 134.62 0) (unit 1)
+    (in_bom yes) (on_board yes) (fields_autoplaced)
+    (property "Reference" "J1" (id 0) (at 24.13 121.92 0)
+      (effects (font (size 1.524 1.524)))
+    )
+    (property "Value" "Power_inlet_vertical" (id 1) (at 24.13 125.73 0)
+      (effects (font (size 1.524 1.524)))
+    )
+    (property "Footprint" "footprints:Wurth-694106402002" (id 2) (at 24.13 129.54 0)
+      (effects (font (size 1.524 1.524)))
+    )
+    (property "Datasheet" "https://www.we-online.com/katalog/datasheet/6941xx402002.pdf" (id 3) (at 28.194 146.558 0)
+      (effects (font (size 1.524 1.524)) hide)
+    )
+    (property "MFG" "Wurth" (id 4) (at 26.67 152.4 0)
+      (effects (font (size 1.27 1.27)) hide)
+    )
+    (property "MPN" "694106402002" (id 5) (at 26.67 154.94 0)
+      (effects (font (size 1.27 1.27)) hide)
+    )
+    (property "Digikey PN" "732-5931-ND" (id 6) (at 28.194 160.147 0)
+      (effects (font (size 1.27 1.27)) hide)
+    )
+    (pin "1")
+    (pin "2")
+    (pin "3")
+  )
   (symbol (lib_id "HPS:GND") (at 179.07 128.27 0) (unit 1)
     (in_bom yes) (on_board yes) (fields_autoplaced)
@@
       (reference "H4") (unit 1) (value "MountingHole") (footprint "footprints:MountingHole_3.2mm_M3")
     )
-    (path "/037a8e6d-4abc-4b60-8de6-cb87d7aa4e51"
-      (reference "J1") (unit 1) (value "PJ-102AH") (footprint "footprints:PJ-102AH")
+    (path "/c2b18a7f-9c0e-4d6f-8b15-5f08e5b2d933"
+      (reference "J1") (unit 1) (value "Power_inlet_vertical") (footprint "footprints:Wurth-694106402002")
     )
     (path "/4c37e47c-98bc-4a5e-8ce0-7f67b646829b"
